File: Hardware/VAR-SOM based/TestBoard 1/TestBoard 1.kicad_sch (KiCad schematic)
At the start: 0 parts

Commit message: Hopeless suggestion from Claude
Other:
- added sheet Gigabit Ethernet (KSZ9031 RGMII PHY + MagJack) (Ethernet.kicad_sch)
- added sheet I2C / SPI / microSD / RGB LEDs / debug UART (Peripherals.kicad_sch)
- added sheet Power input / regulators / status LEDs (Power.kicad_sch)
- added sheet Raspberry Pi 40-pin HAT header (J9) (RPi_Header.kicad_sch)
- added sheet SoM Connector (VAR-SOM-MX8M-PLUS) (SOM.kicad_sch)
- added sheet USB 2.0 host ports (front + back) (USB.kicad_sch)
- note added: "3x addressable RGB LEDs. 4-layer PCB, whole-mm outline, 4x M3 mounting holes 4mm from edges."
- note added: "Ethernet (back), 2x USB2.0-A host (front+back), I2C & 2x SPI IDC, microSD (front),"
- note added: "Proof-of-concept carrier for the Flux project. Features per Readme.md:"
- note added: "RPi 40-pin HAT header, 12V input with on-board 5V/3V3 regulators, power status LEDs,"
- note added: "TestBoard1 : VAR-SOM-MX8M-PLUS proof-of-concept carrier"
- company: (none) -> OpenTools / Flux
- title: (none) -> TestBoard1 - VAR-SOM-MX8M-PLUS carrier (root)
Changed lines of the file:
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@@
 	(generator "eeschema")
 	(generator_version "10.0")
-	(paper "A4")
+	(paper "A3")
+	(title_block
+		(title "TestBoard1 - VAR-SOM-MX8M-PLUS carrier (root)")
+		(rev "A")
+		(company "OpenTools / Flux")
+	)
+	(text "TestBoard1 : VAR-SOM-MX8M-PLUS proof-of-concept carrier" (at 25.4 25.4 0) (effects (font (size 3.0 3.0) (bold yes)) (justify left)))
+	(text "Proof-of-concept carrier for the Flux project. Features per Readme.md:" (at 25.4 170.0 0) (effects (font (size 2.0 2.0)) (justify left)))
+	(text "Ethernet (back), 2x USB2.0-A host (front+back), I2C & 2x SPI IDC, microSD (front)," (at 25.4 176.0 0) (effects (font (size 2.0 2.0)) (justify left)))
+	(text "RPi 40-pin HAT header, 12V input with on-board 5V/3V3 regulators, power status LEDs," (at 25.4 182.0 0) (effects (font (size 2.0 2.0)) (justify left)))
+	(text "3x addressable RGB LEDs. 4-layer PCB, whole-mm outline, 4x M3 mounting holes 4mm from edges." (at 25.4 188.0 0) (effects (font (size 2.0 2.0)) (justify left)))
+	(sheet (at 25.40 38.00) (size 63.5 33.02)
+		(fields_autoplaced yes)
+		(stroke (width 0.1524) (type solid))
+		(fill (color 0 0 0 0.0))
+		(property "Sheetname" "SoM Connector (VAR-SOM-MX8M-PLUS)" (at 25.40 37.00 0) (effects (font (size 1.6 1.6)) (justify left bottom)))
+		(property "Sheetfile" "SOM.kicad_sch" (at 25.40 72.50 0) (effects (font (size 1.27 1.27)) (justify left top)))
+		(instances (project "TestBoard 1" (path "/ea2adde5-c377-cb5e-09d1-4b71935c6f32" (page "2"))))
+	)
+	(sheet (at 114.30 38.00) (size 63.5 33.02)
+		(fields_autoplaced yes)
+		(stroke (width 0.1524) (type solid))
+		(fill (color 0 0 0 0.0))
+		(property "Sheetname" "Power input / regulators / status LEDs" (at 114.30 37.00 0) (effects (font (size 1.6 1.6)) (justify left bottom)))
+		(property "Sheetfile" "Power.kicad_sch" (at 114.30 72.50 0) (effects (font (size 1.27 1.27)) (justify left top)))
+		(instances (project "TestBoard 1" (path "/ea2adde5-c377-cb5e-09d1-4b71935c6f32" (page "3"))))
+	)
+	(sheet (at 203.20 38.00) (size 63.5 33.02)
+		(fields_autoplaced yes)
+		(stroke (width 0.1524) (type solid))
+		(fill (color 0 0 0 0.0))
+		(property "Sheetname" "Gigabit Ethernet (KSZ9031 RGMII PHY + MagJack)" (at 203.20 37.00 0) (effects (font (size 1.6 1.6)) (justify left bottom)))
+		(property "Sheetfile" "Ethernet.kicad_sch" (at 203.20 72.50 0) (effects (font (size 1.27 1.27)) (justify left top)))
+		(instances (project "TestBoard 1" (path "/ea2adde5-c377-cb5e-09d1-4b71935c6f32" (page "4"))))
+	)
+	(sheet (at 25.40 88.80) (size 63.5 33.02)
+		(fields_autoplaced yes)
+		(stroke (width 0.1524) (type solid))
+		(fill (color 0 0 0 0.0))
+		(property "Sheetname" "USB 2.0 host ports (front + back)" (at 25.40 87.80 0) (effects (font (size 1.6 1.6)) (justify left bottom)))
+		(property "Sheetfile" "USB.kicad_sch" (at 25.40 123.30 0) (effects (font (size 1.27 1.27)) (justify left top)))
+		(instances (project "TestBoard 1" (path "/ea2adde5-c377-cb5e-09d1-4b71935c6f32" (page "5"))))
+	)
+	(sheet (at 114.30 88.80) (size 63.5 33.02)
+		(fields_autoplaced yes)
+		(stroke (width 0.1524) (type solid))
+		(fill (color 0 0 0 0.0))
+		(property "Sheetname" "I2C / SPI / microSD / RGB LEDs / debug UART" (at 114.30 87.80 0) (effects (font (size 1.6 1.6)) (justify left bottom)))
+		(property "Sheetfile" "Peripherals.kicad_sch" (at 114.30 123.30 0) (effects (font (size 1.27 1.27)) (justify left top)))
+		(instances (project "TestBoard 1" (path "/ea2adde5-c377-cb5e-09d1-4b71935c6f32" (page "6"))))
+	)
+	(sheet (at 203.20 88.80) (size 63.5 33.02)
+		(fields_autoplaced yes)
+		(stroke (width 0.1524) (type solid))
+		(fill (color 0 0 0 0.0))
+		(property "Sheetname" "Raspberry Pi 40-pin HAT header (J9)" (at 203.20 87.80 0) (effects (font (size 1.6 1.6)) (justify left bottom)))
+		(property "Sheetfile" "RPi_Header.kicad_sch" (at 203.20 123.30 0) (effects (font (size 1.27 1.27)) (justify left top)))
+		(instances (project "TestBoard 1" (path "/ea2adde5-c377-cb5e-09d1-4b71935c6f32" (page "7"))))
+	)
 	(sheet_instances
-		(path "/"
-			(page "1")
-		)
+		(path "/" (page "1"))
+		(path "/ddca7cf4-2b3e-5b0b-6469-47bfec6efb30" (page "2"))
+		(path "/6d9eefb8-8bf1-4076-8431-4e974facd3cc" (page "3"))
+		(path "/07a642bd-7df0-bcee-30b3-c3281461ebfb" (page "4"))
+		(path "/a56ce177-900e-77b6-63a0-aa93ead67f5e" (page "5"))
+		(path "/c0e98371-a9c9-10f9-b5ce-24a42434225b" (page "6"))
+		(path "/1857ca50-ddcf-4bad-bbc2-b46409be2a84" (page "7"))
 	)
 	(embedded_fonts no)
